Commit message: added gnss, imu and hardware interfaces

File: amr_sweeper_description/urdf/control/odrive_ros2_control.xacro (robot description, xacro)
@@ -1,4 +1,5 @@
 <?xml version="1.0"?>
 <robot xmlns:xacro="http://www.ros.org/wiki/xacro">
+<!--     Real Robot     -->
   <xacro:unless value="$(arg sim_mode)">
     <ros2_control name="RealRobot" type="system">
@@ -8,13 +9,28 @@
       </hardware>
       <joint name="LeftWheel_joint">
+        <command_interface name="velocity">
+          <param name="min">-10</param>
+          <param name="max">10</param>
+        </command_interface>
+        <state_interface name="velocity"/>
+        <state_interface name="position"/>
         <param name="node_id">0</param>
         <param name="gear_ratio">50.0</param>
+        <param name="motor_direction">CCW</param>
       </joint>
       <joint name="RightWheel_joint">
+        <command_interface name="velocity">
+          <param name="min">-10</param>
+          <param name="max">10</param>
+        </command_interface>
+        <state_interface name="velocity"/>
+        <state_interface name="position"/>
         <param name="node_id">2</param>
         <param name="gear_ratio">50.0</param>
+        <param name="motor_direction">CW</param>
       </joint>
     </ros2_control>
   </xacro:unless>
+<!--     Simulation     -->
   <xacro:if value="$(arg sim_mode)">
     <ros2_control name="GazeboSystem" type="system">

File: amr_sweeper_description/urdf/robot/robot_core.xacro (robot description, xacro)
@@ -9,11 +9,5 @@
     <origin xyz="0 0 0.13" rpy="0 ${base_pitch_rad} 0"/>
   </joint>
-  <link name="base_link"/>
-  <joint name="chassis_joint" type="fixed">
-    <parent link="base_link"/>
-    <child link="chassis_link"/>
-    <origin xyz="0 0 0" rpy="0 0 0"/>
-  </joint>
-  <link name="chassis_link">
+  <link name="base_link">
     <visual>
       <origin xyz="0 0 0" rpy="0 0 0"/>

Commit message: Update

File: amr_sweeper_description/urdf/control/odrive_ros2_control.xacro (robot description, xacro)
@@ -1,74 +1,31 @@
 <?xml version="1.0"?>
 <robot xmlns:xacro="http://www.ros.org/wiki/xacro">
-<!--     Real Robot     -->
-  <xacro:unless value="$(arg sim_mode)">
-    <ros2_control name="RealRobot" type="system">
-      <hardware>
-        <plugin>odrive_ros2_control_plugin/ODriveHardwareInterface</plugin>
-        <param name="can">can0</param>
-      </hardware>
-      <joint name="LeftWheel_joint">
-        <command_interface name="velocity">
-          <param name="min">-10</param>
-          <param name="max">10</param>
-        </command_interface>
-        <state_interface name="velocity"/>
-        <state_interface name="position"/>
-        <param name="node_id">0</param>
-        <param name="gear_ratio">50.0</param>
-        <param name="motor_direction">CCW</param>
-      </joint>
-      <joint name="RightWheel_joint">
-        <command_interface name="velocity">
-          <param name="min">-10</param>
-          <param name="max">10</param>
-        </command_interface>
-        <state_interface name="velocity"/>
-        <state_interface name="position"/>
-        <param name="node_id">2</param>
-        <param name="gear_ratio">50.0</param>
-        <param name="motor_direction">CW</param>
-      </joint>
-    </ros2_control>
-  </xacro:unless>
-<!--     Simulation     -->
-  <xacro:if value="$(arg sim_mode)">
-    <ros2_control name="GazeboSystem" type="system">
-      <hardware>
-        <plugin>gz_ros2_control/GazeboSimSystem</plugin>
-      </hardware>
-      <joint name="LeftWheel_joint">
-        <command_interface name="velocity">
-          <param name="min">-10</param>
-          <param name="max">10</param>
-        </command_interface>
-        <state_interface name="velocity"/>
-        <state_interface name="position"/>
-      </joint>
-      <joint name="RightWheel_joint">
-        <command_interface name="velocity">
-          <param name="min">-10</param>
-          <param name="max">10</param>
-        </command_interface>
-        <state_interface name="velocity"/>
-        <state_interface name="position"/>
-      </joint>
-      <joint name="LeftBrush_joint">
-        <command_interface name="velocity">
-          <param name="min">-10</param>
-          <param name="max">10</param>
-        </command_interface>
-        <state_interface name="velocity"/>
-        <state_interface name="position"/>
-      </joint>
-      <joint name="RightBrush_joint">
-        <command_interface name="velocity">
-          <param name="min">-10</param>
-          <param name="max">10</param>
-        </command_interface>
-        <state_interface name="velocity"/>
-        <state_interface name="position"/>
-      </joint>
-    </ros2_control>
-  </xacro:if>
+  <ros2_control name="RealRobot" type="system">
+    <hardware>
+      <plugin>odrive_ros2_control_plugin/ODriveHardwareInterface</plugin>
+      <param name="can">can0</param>
+    </hardware>
+    <joint name="LeftWheel_joint">
+      <command_interface name="velocity">
+        <param name="min">-10</param>
+        <param name="max">10</param>
+      </command_interface>
+      <state_interface name="velocity"/>
+      <state_interface name="position"/>
+      <param name="node_id">0</param>
+      <param name="gear_ratio">50.0</param>
+      <param name="motor_direction">CCW</param>
+    </joint>
+    <joint name="RightWheel_joint">
+      <command_interface name="velocity">
+        <param name="min">-10</param>
+        <param name="max">10</param>
+      </command_interface>
+      <state_interface name="velocity"/>
+      <state_interface name="position"/>
+      <param name="node_id">2</param>
+      <param name="gear_ratio">50.0</param>
+      <param name="motor_direction">CW</param>
+    </joint>
+  </ros2_control>
 </robot>

File: amr_sweeper_description/urdf/control/steadydrive_ros2_control.xacro (robot description, xacro)
@@ -1,24 +1,22 @@
 <?xml version="1.0"?>
 <robot xmlns:xacro="http://www.ros.org/wiki/xacro" name="robot">
-  <xacro:unless value="$(arg sim_mode)">
-    <ros2_control name="steadydrive_ros2_control" type="system">
-      <hardware>
-        <plugin>steadydrive_hw_interface/SteadydriveHardwareInterface</plugin>
-        <param name="topic_speed_output_left">steadydrive_left/speed_control</param>
-        <param name="topic_speed_output_right">steadydrive_right/speed_control</param>
-        <param name="topic_motor_state_left">steadydrive_left/joint_state</param>
-        <param name="topic_motor_state_right">steadydrive_right/joint_state</param>
-      </hardware>
-      <joint name="LeftBrush_joint">
-        <command_interface name="velocity"/>
-        <state_interface name="velocity"/>
-        <state_interface name="position"/>
-      </joint>
-      <joint name="RightBrush_joint">
-        <command_interface name="velocity"/>
-        <state_interface name="velocity"/>
-        <state_interface name="position"/>
-      </joint>
-    </ros2_control>
-  </xacro:unless>
+  <ros2_control name="steadydrive_ros2_control" type="system">
+    <hardware>
+      <plugin>steadydrive_hw_interface/SteadydriveHardwareInterface</plugin>
+      <param name="topic_speed_output_left">steadydrive_left/speed_control</param>
+      <param name="topic_speed_output_right">steadydrive_right/speed_control</param>
+      <param name="topic_motor_state_left">steadydrive_left/joint_state</param>
+      <param name="topic_motor_state_right">steadydrive_right/joint_state</param>
+    </hardware>
+    <joint name="LeftBrush_joint">
+      <command_interface name="velocity"/>
+      <state_interface name="velocity"/>
+      <state_interface name="position"/>
+    </joint>
+    <joint name="RightBrush_joint">
+      <command_interface name="velocity"/>
+      <state_interface name="velocity"/>
+      <state_interface name="position"/>
+    </joint>
+  </ros2_control>
 </robot>

File: amr_sweeper_description/urdf/robot/robot.urdf.xacro (robot description, xacro)
@@ -2,5 +2,4 @@
 <robot xmlns:xacro="http://www.ros.org/wiki/xacro" name="amr_sweeper">
   <xacro:arg name="use_ros2_control" default="true"/>
-  <xacro:arg name="sim_mode" default="false"/>
   <xacro:arg name="enable_top_cameras" default="true"/>
   <xacro:arg name="enable_gnss" default="true"/>
@@ -25,6 +24,3 @@
     <xacro:include filename="$(find amr_sweeper_description)/urdf/control/steadydrive_ros2_control.xacro"/>
   </xacro:if>
-  <xacro:unless value="$(arg use_ros2_control)">
-    <xacro:include filename="$(find amr_sweeper_description)/urdf/control/gazebo_control.xacro"/>
-  </xacro:unless>
 </robot>

File: amr_sweeper_description/urdf/sensors/GNSS_sensor.xacro (robot description, xacro)
@@ -15,31 +15,3 @@
     </visual>
   </link>
-  <xacro:if value="$(arg sim_mode)">
-    <gazebo reference="gnss_link">
-      <sensor name="gnss_sensor" type="navsat">
-        <always_on>true</always_on>
-        <update_rate>1.0</update_rate>
-        <topic>gnss/navsat</topic>
-        <navsat>
-          <position_sensing>
-            <horizontal>
-              <noise type="gaussian">
-                <mean>0.00001</mean>
-                <stddev>0.00001</stddev>
-              </noise>
-            </horizontal>
-          </position_sensing>
-          <velocity_sensing>
-            <horizontal>
-              <noise type="gaussian">
-                <mean>0.0</mean>
-                <stddev>0.00001</stddev>
-              </noise>
-            </horizontal>
-          </velocity_sensing>
-        </navsat>
-        <plugin filename="gz-sim-navsat-system" name="gz::sim::systems::NavSat"/>
-      </sensor>
-    </gazebo>
-  </xacro:if>
 </robot>

File: amr_sweeper_description/urdf/sensors/IMU_sensor.xacro (robot description, xacro)
@@ -7,14 +7,3 @@
   </joint>
   <link name="imu_link"/>
-  <xacro:if value="$(arg sim_mode)">
-    <gazebo reference="imu_link">
-      <sensor name="imu_sensor" type="imu">
-        <always_on>true</always_on>
-        <update_rate>10</update_rate>
-        <visualize>true</visualize>
-        <topic>imu/data</topic>
-        <plugin filename="gz-sim-imu-system" name="gz::sim::systems::Imu"/>
-      </sensor>
-    </gazebo>
-  </xacro:if>
 </robot>

File: amr_sweeper_description/urdf/sensors/depth_camera.xacro (robot description, xacro)
@@ -49,44 +49,3 @@
   </joint>
   <link name="camera_link_optical"/>
-  <xacro:if value="$(arg sim_mode)">
-    <gazebo reference="camera_link">
-      <sensor name="depth_camera" type="depth_camera">
-        <update_rate>10</update_rate>
-        <topic>depth_camera</topic>
-        <camera>
-          <horizontal_fov>1.05</horizontal_fov>
-          <image>
-            <width>256</width>
-            <height>256</height>
-            <format>R_FLOAT32</format>
-          </image>
-          <clip>
-            <near>0.1</near>
-            <far>10.0</far>
-          </clip>
-        </camera>
-      </sensor>
-    </gazebo>
-    <gazebo reference="camera_link">
-      <sensor name="camera" type="camera">
-        <pose>0 0 0 0 0 0</pose>
-        <visualize>true</visualize>
-        <update_rate>10</update_rate>
-        <camera>
-          <camera_info_topic>camera/camera_info</camera_info_topic>
-          <horizontal_fov>1.089</horizontal_fov>
-          <image>
-            <format>R8G8B8</format>
-            <width>640</width>
-            <height>480</height>
-          </image>
-          <clip>
-            <near>0.05</near>
-            <far>8.0</far>
-          </clip>
-        </camera>
-        <topic>camera/image_raw</topic>
-      </sensor>
-    </gazebo>
-  </xacro:if>
 </robot>
