Commit message: fixing tool position

File: amr_sweeper_description/urdf/control/steadydrive_ros2_control.xacro (robot description, xacro)
@@ -13,5 +13,5 @@
       <state_interface name="position"/>
       <state_interface name="velocity"/>
-      <param name="gear_ratio">1.0</param>
+      <param name="gear_ratio">10.0</param>
       <param name="positive_motor_direction">CCW</param>
     </joint>

File: amr_sweeper_description/urdf/robot/robot_core.xacro (robot description, xacro)
@@ -112,9 +112,9 @@
     <origin xyz="0 0.155 -0.08" rpy="0 0 0"/>
     <parent link="tool_link"/>
-    <child link="left_brush_link"/>
+    <child link="left_tool_link"/>
     <axis xyz="0 0 1"/>
     <dynamics damping="0.02" friction="0.02"/>
   </joint>
-  <link name="left_brush_link">
+  <link name="left_tool_link">
     <visual>
       <origin xyz="0 0 0" rpy="0 0 0"/>
@@ -139,9 +139,9 @@
     <origin xyz="0 -0.155 -0.08" rpy="0 0 0"/>
     <parent link="tool_link"/>
-    <child link="right_brush_link"/>
+    <child link="right_tool_link"/>
     <axis xyz="0 0 1"/>
     <dynamics damping="0.02" friction="0.02"/>
   </joint>
-  <link name="right_brush_link">
+  <link name="right_tool_link">
     <visual>
       <origin xyz="0 0 0" rpy="0 0 0"/>
