Commit message: Added correction for using internal IMU.

File: amr_sweeper_description/urdf/sensors/depth_camera.xacro (robot description, xacro)
@@ -59,4 +59,10 @@
   </joint>
   <link name="depth_camera_imu_frame"/>
+  <joint name="depth_camera_motion_optical_joint" type="fixed">
+    <parent link="depth_camera_imu_frame"/>
+    <child link="depth_camera_motion_optical_frame"/>
+    <origin xyz="0 0 0" rpy="${-pi/2} 0 ${-pi/2}"/>
+  </joint>
+  <link name="depth_camera_motion_optical_frame"/>
   <joint name="depth_camera_depth_optical_joint" type="fixed">
     <parent link="depth_camera_depth_frame"/>
