Commit message: Implemented 180deg yaw offset in IMU driver

File: amr_sweeper_description/urdf/sensors/IMU_sensor.xacro (robot description, xacro)
@@ -4,5 +4,5 @@
     <parent link="base_link"/>
     <child link="imu_link"/>
-    <origin xyz="0.088 0.0 0.184" rpy="0 0 ${pi}"/>
+    <origin xyz="0.088 0.0 0.184" rpy="0 0 0"/>
   </joint>
   <link name="imu_link"/>

Commit message: Update IMU_sensor.xacro

File: amr_sweeper_description/urdf/sensors/IMU_sensor.xacro (robot description, xacro)
@@ -4,5 +4,5 @@
     <parent link="base_link"/>
     <child link="imu_link"/>
-    <origin xyz="0.088 0.0 0.184" rpy="0 0 0"/>
+    <origin xyz="0.088 0.0 0.184" rpy="0 0 ${-pi/2}"/>
   </joint>
   <link name="imu_link"/>

Commit message: Update IMU_sensor.xacro

File: amr_sweeper_description/urdf/sensors/IMU_sensor.xacro (robot description, xacro)
@@ -4,5 +4,5 @@
     <parent link="base_link"/>
     <child link="imu_link"/>
-    <origin xyz="0.088 0.0 0.184" rpy="0 0 ${-pi/2}"/>
+    <origin xyz="0.088 0.0 0.184" rpy="0 0 ${pi}"/>
   </joint>
   <link name="imu_link"/>

Commit message: imu

File: amr_sweeper_description/urdf/sensors/IMU_sensor.xacro (robot description, xacro)
@@ -4,5 +4,5 @@
     <parent link="base_link"/>
     <child link="imu_link"/>
-    <origin xyz="0.088 0.0 0.184" rpy="0 0 ${pi}"/>
+    <origin xyz="0.088 0.0 0.184" rpy="0 0 0/>
   </joint>
   <link name="imu_link"/>

Commit message: Update IMU_sensor.xacro

File: amr_sweeper_description/urdf/sensors/IMU_sensor.xacro (robot description, xacro)
@@ -4,5 +4,5 @@
     <parent link="base_link"/>
     <child link="imu_link"/>
-    <origin xyz="0.088 0.0 0.184" rpy="0 0 0/>
+    <origin xyz="0.088 0.0 0.184" rpy="0 0 0"/>
   </joint>
   <link name="imu_link"/>
