Commit message: Update robot_core.xacro

File: amr_sweeper_description/urdf/robot/robot_core.xacro (robot description, xacro)
@@ -1,11 +1,25 @@
 <?xml version="1.0"?>
 <robot xmlns:xacro="http://www.ros.org/wiki/xacro">
-  <xacro:property name="base_pitch_deg" value="0.0"/>
-  <xacro:property name="base_pitch_rad" value="${base_pitch_deg * pi / 180.0}"/>
   <link name="base_footprint"/>
-  <joint name="base_footprint_joint" type="fixed">
+  <link name="base_roll_link"/>
+  <joint name="base_roll_joint" type="revolute">
     <parent link="base_footprint"/>
+    <child link="base_roll_link"/>
+    <origin xyz="0 0 0.13" rpy="0 0 0"/>
+    <axis xyz="1 0 0"/>
+    <limit lower="-3.141592653589793" upper="3.141592653589793" effort="1.0" velocity="10.0"/>
+  </joint>
+  <link name="base_pitch_link"/>
+  <joint name="base_pitch_joint" type="revolute">
+    <parent link="base_roll_link"/>
+    <child link="base_pitch_link"/>
+    <origin xyz="0 0 0" rpy="0 0 0"/>
+    <axis xyz="0 1 0"/>
+    <limit lower="-3.141592653589793" upper="3.141592653589793" effort="1.0" velocity="10.0"/>
+  </joint>
+  <joint name="base_link_mount_joint" type="fixed">
+    <parent link="base_pitch_link"/>
     <child link="base_link"/>
-    <origin xyz="0 0 0.13" rpy="0 ${base_pitch_rad} 0"/>
+    <origin xyz="0 0 0" rpy="0 0 0"/>
   </joint>
   <link name="base_link">

Commit message: Commented out frames between base_link and base_footprint. Applied tilt to IMU

File: amr_sweeper_description/urdf/robot/robot_core.xacro (robot description, xacro)
@@ -2,5 +2,5 @@
 <robot xmlns:xacro="http://www.ros.org/wiki/xacro">
   <link name="base_footprint"/>
-  <link name="base_roll_link"/>
+  <!--link name="base_roll_link"/>
   <joint name="base_roll_joint" type="revolute">
     <parent link="base_footprint"/>
@@ -20,4 +20,9 @@
   <joint name="base_link_mount_joint" type="fixed">
     <parent link="base_pitch_link"/>
+    <child link="base_link"/>
+    <origin xyz="0 0 0" rpy="0 0 0"/>
+  </joint-->
+  <joint name="base_footprint_to_base_link" type="fixed">
+    <parent link="base_footprint"/>
     <child link="base_link"/>
     <origin xyz="0 0 0" rpy="0 0 0"/>

File: amr_sweeper_description/urdf/sensors/IMU_sensor.xacro (robot description, xacro)
@@ -4,5 +4,5 @@
     <parent link="base_link"/>
     <child link="imu_link"/>
-    <origin xyz="0.088 0.0 0.184" rpy="0 0 0"/>
+    <origin xyz="0.088 0.0 0.184" rpy="0 0.06353 0"/>
   </joint>
   <link name="imu_link"/>

Commit message: removed dynamic joints

File: amr_sweeper_description/urdf/robot/robot_core.xacro (robot description, xacro)
@@ -1,26 +1,4 @@
 <?xml version="1.0"?>
 <robot xmlns:xacro="http://www.ros.org/wiki/xacro">
-  <link name="base_footprint"/>
-  <link name="base_roll_link"/>
-  <joint name="base_roll_joint" type="revolute">
-    <parent link="base_footprint"/>
-    <child link="base_roll_link"/>
-    <origin xyz="0 0 0.13" rpy="0 0 0"/>
-    <axis xyz="1 0 0"/>
-    <limit lower="-3.141592653589793" upper="3.141592653589793" effort="1.0" velocity="10.0"/>
-  </joint>
-  <link name="base_pitch_link"/>
-  <joint name="base_pitch_joint" type="revolute">
-    <parent link="base_roll_link"/>
-    <child link="base_pitch_link"/>
-    <origin xyz="0 0 0" rpy="0 0 0"/>
-    <axis xyz="0 1 0"/>
-    <limit lower="-3.141592653589793" upper="3.141592653589793" effort="1.0" velocity="10.0"/>
-  </joint>
-  <joint name="base_link_mount_joint" type="fixed">
-    <parent link="base_pitch_link"/>
-    <child link="base_link"/>
-    <origin xyz="0 0 0" rpy="0 0 0"/>
-  </joint>
   <link name="base_link">
     <visual>

Commit message: updated bug

File: amr_sweeper_description/urdf/robot/robot_core.xacro (robot description, xacro)
@@ -1,4 +1,10 @@
 <?xml version="1.0"?>
 <robot xmlns:xacro="http://www.ros.org/wiki/xacro">
+  <link name="base_root"/>
+  <joint name="base_root_to_base_link" type="fixed">
+    <parent link="base_root"/>
+    <child link="base_link"/>
+    <origin xyz="0 0 0" rpy="0 0 0"/>
+  </joint>
   <link name="base_link">
     <visual>

Commit message: Update robot_core.xacro

File: amr_sweeper_description/urdf/robot/robot_core.xacro (robot description, xacro)
@@ -2,8 +2,14 @@
 <robot xmlns:xacro="http://www.ros.org/wiki/xacro">
   <link name="base_root"/>
-  <joint name="base_root_to_base_link" type="fixed">
+  <link name="base_footprint"/>
+  <joint name="base_root_to_base_footprint" type="fixed">
     <parent link="base_root"/>
+    <child link="base_footprint"/>
+    <origin xyz="0 0 0" rpy="0 0 0"/>
+  </joint>
+  <joint name="base_footprint_to_base_link" type="fixed">
+    <parent link="base_footprint"/>
     <child link="base_link"/>
-    <origin xyz="0 0 0" rpy="0 0 0"/>
+    <origin xyz="0 0 0.13" rpy="0 0 0"/>
   </joint>
   <link name="base_link">

Commit message: Update robot_core.xacro

File: amr_sweeper_description/urdf/robot/robot_core.xacro (robot description, xacro)
@@ -2,14 +2,8 @@
 <robot xmlns:xacro="http://www.ros.org/wiki/xacro">
   <link name="base_root"/>
-  <link name="base_footprint"/>
-  <joint name="base_root_to_base_footprint" type="fixed">
+  <joint name="base_root_to_base_link" type="fixed">
     <parent link="base_root"/>
-    <child link="base_footprint"/>
+    <child link="base_link"/>
     <origin xyz="0 0 0" rpy="0 0 0"/>
-  </joint>
-  <joint name="base_footprint_to_base_link" type="fixed">
-    <parent link="base_footprint"/>
-    <child link="base_link"/>
-    <origin xyz="0 0 0.13" rpy="0 0 0"/>
   </joint>
   <link name="base_link">

Commit message: Update robot_core.xacro

File: amr_sweeper_description/urdf/robot/robot_core.xacro (robot description, xacro)
@@ -1,10 +1,4 @@
 <?xml version="1.0"?>
 <robot xmlns:xacro="http://www.ros.org/wiki/xacro">
-  <link name="base_root"/>
-  <joint name="base_root_to_base_link" type="fixed">
-    <parent link="base_root"/>
-    <child link="base_link"/>
-    <origin xyz="0 0 0" rpy="0 0 0"/>
-  </joint>
   <link name="base_link">
     <visual>

Commit message: Update robot_core.xacro

File: amr_sweeper_description/urdf/robot/robot_core.xacro (robot description, xacro)
@@ -2,4 +2,11 @@
 <robot xmlns:xacro="http://www.ros.org/wiki/xacro">
   <link name="base_link">
+  </link>
+  <joint name="base_link_to_chassis_link" type="fixed">
+    <parent link="base_link"/>
+    <child link="chassis_link"/>
+    <origin xyz="0 0 0" rpy="0 0 0"/>
+  </joint>
+  <link name="chassis_link">
     <visual>
       <origin xyz="0 0 0" rpy="0 0 0"/>
