Commit message: Update robot_core.xacro

File: amr_sweeper_description/urdf/robot/robot_core.xacro (robot description, xacro)
@@ -39,5 +39,5 @@
         <origin xyz="0.06 0.0 0.095" rpy="0 0 0"/>
         <geometry>
-          <box size="0.70 0.55 0.24"/>
+          <box size="0.70 0.40 0.24"/>
         </geometry>
       </collision>
@@ -70,10 +70,20 @@
       <material name="yellow"/>
     </visual>
-    <collision>
-      <origin xyz="0 0 0" rpy="${pi/2} 0 0"/>
-      <geometry>
-        <mesh filename="package://amr_sweeper_description/meshes/WheelAssembly.stl"/>
-      </geometry>
-    </collision>
+    <xacro:if value="$(arg simulation_physics)">
+      <collision>
+        <origin xyz="0 0 0" rpy="0 0 0"/>
+        <geometry>
+          <cylinder radius="0.13" length="0.08"/>
+        </geometry>
+      </collision>
+    </xacro:if>
+    <xacro:unless value="$(arg simulation_physics)">
+      <collision>
+        <origin xyz="0 0 0" rpy="${pi/2} 0 0"/>
+        <geometry>
+          <mesh filename="package://amr_sweeper_description/meshes/WheelAssembly.stl"/>
+        </geometry>
+      </collision>
+    </xacro:unless>
     <inertial>
       <origin xyz="0 -0.000056 0" rpy="0 0 0"/>
@@ -96,10 +106,20 @@
       <material name="yellow"/>
     </visual>
-    <collision>
-      <origin xyz="0 0 0" rpy="${pi/2} 0 0"/>
-      <geometry>
-        <mesh filename="package://amr_sweeper_description/meshes/WheelAssembly.stl"/>
-      </geometry>
-    </collision>
+    <xacro:if value="$(arg simulation_physics)">
+      <collision>
+        <origin xyz="0 0 0" rpy="0 0 0"/>
+        <geometry>
+          <cylinder radius="0.13" length="0.08"/>
+        </geometry>
+      </collision>
+    </xacro:if>
+    <xacro:unless value="$(arg simulation_physics)">
+      <collision>
+        <origin xyz="0 0 0" rpy="${pi/2} 0 0"/>
+        <geometry>
+          <mesh filename="package://amr_sweeper_description/meshes/WheelAssembly.stl"/>
+        </geometry>
+      </collision>
+    </xacro:unless>
     <inertial>
       <origin xyz="0 0.000056 0" rpy="0 0 0"/>
@@ -143,10 +163,20 @@
       <material name="red"/>
     </visual>
-    <collision>
-      <origin xyz="0 0 0" rpy="0 0 0"/>
-      <geometry>
-        <mesh filename="package://amr_sweeper_description/meshes/Brush.stl"/>
-      </geometry>
-    </collision>
+    <xacro:if value="$(arg simulation_physics)">
+      <collision>
+        <origin xyz="0 0 -0.055" rpy="0 0 0"/>
+        <geometry>
+          <cylinder radius="0.14" length="0.04"/>
+        </geometry>
+      </collision>
+    </xacro:if>
+    <xacro:unless value="$(arg simulation_physics)">
+      <collision>
+        <origin xyz="0 0 0" rpy="0 0 0"/>
+        <geometry>
+          <mesh filename="package://amr_sweeper_description/meshes/Brush.stl"/>
+        </geometry>
+      </collision>
+    </xacro:unless>
     <inertial>
       <origin xyz="0.000007 0 -0.00877" rpy="0 0 0"/>
@@ -170,10 +200,20 @@
       <material name="red"/>
     </visual>
-    <collision>
-      <origin xyz="0 0 0" rpy="0 0 0"/>
-      <geometry>
-        <mesh filename="package://amr_sweeper_description/meshes/Brush.stl"/>
-      </geometry>
-    </collision>
+    <xacro:if value="$(arg simulation_physics)">
+      <collision>
+        <origin xyz="0 0 -0.055" rpy="0 0 0"/>
+        <geometry>
+          <cylinder radius="0.14" length="0.04"/>
+        </geometry>
+      </collision>
+    </xacro:if>
+    <xacro:unless value="$(arg simulation_physics)">
+      <collision>
+        <origin xyz="0 0 0" rpy="0 0 0"/>
+        <geometry>
+          <mesh filename="package://amr_sweeper_description/meshes/Brush.stl"/>
+        </geometry>
+      </collision>
+    </xacro:unless>
     <inertial>
       <origin xyz="0.000007 0 -0.00877" rpy="0 0 0"/>
