Commit message: added simulations

File: amr_sweeper_description/urdf/robot/robot.urdf.xacro (robot description, xacro)
@@ -2,4 +2,6 @@
 <robot xmlns:xacro="http://www.ros.org/wiki/xacro" name="amr_sweeper">
   <xacro:arg name="use_ros2_control" default="true"/>
+  <xacro:arg name="use_simulation" default="false"/>
+  <xacro:arg name="simulation_physics" default="false"/>
   <xacro:arg name="robot_namespace" default="amr_sweeper"/>
   <xacro:arg name="enable_usb_cameras" default="true"/>
@@ -22,6 +24,12 @@
   </xacro:if>
   <xacro:if value="$(arg use_ros2_control)">
-    <xacro:include filename="$(find amr_sweeper_description)/urdf/control/odrive_ros2_control.xacro"/>
-    <xacro:include filename="$(find amr_sweeper_description)/urdf/control/steadydrive_ros2_control.xacro"/>
+    <xacro:if value="$(arg use_simulation)">
+      <xacro:include filename="$(find amr_sweeper_description)/urdf/control/odrive_ros2_control_sim.xacro"/>
+      <xacro:include filename="$(find amr_sweeper_description)/urdf/control/steadydrive_ros2_control_sim.xacro"/>
+    </xacro:if>
+    <xacro:unless value="$(arg use_simulation)">
+      <xacro:include filename="$(find amr_sweeper_description)/urdf/control/odrive_ros2_control.xacro"/>
+      <xacro:include filename="$(find amr_sweeper_description)/urdf/control/steadydrive_ros2_control.xacro"/>
+    </xacro:unless>
   </xacro:if>
 </robot>

File: amr_sweeper_description/urdf/robot/robot_core.xacro (robot description, xacro)
@@ -2,4 +2,23 @@
 <robot xmlns:xacro="http://www.ros.org/wiki/xacro">
   <link name="base_link">
+    <xacro:if value="$(arg simulation_physics)">
+      <visual>
+        <origin xyz="0 0 0" rpy="0 0 0"/>
+        <geometry>
+          <box size="0.01 0.01 0.01"/>
+        </geometry>
+      </visual>
+      <collision>
+        <origin xyz="0 0 0" rpy="0 0 0"/>
+        <geometry>
+          <box size="0.01 0.01 0.01"/>
+        </geometry>
+      </collision>
+      <inertial>
+        <origin xyz="0 0 0" rpy="0 0 0"/>
+        <mass value="0.01"/>
+        <inertia ixx="1.0e-4" ixy="0.0" ixz="0.0" iyy="1.0e-4" iyz="0.0" izz="1.0e-4"/>
+      </inertial>
+    </xacro:if>
   </link>
   <joint name="base_link_to_chassis_link" type="fixed">
@@ -16,9 +35,24 @@
       <material name="grey"/>
     </visual>
-    <inertial>
-      <origin xyz="0.064266 0.001648 0.095511" rpy="0 0 0"/>
-      <mass value="20.656"/>
-      <inertia ixx="0.110436033" ixy="0.007458962" ixz="-0.047319713" iyy="0.439622462" iyz="0.006320743" izz="0.625226807"/>
-    </inertial>
+    <xacro:if value="$(arg simulation_physics)">
+      <collision>
+        <origin xyz="0.06 0.0 0.095" rpy="0 0 0"/>
+        <geometry>
+          <box size="0.70 0.55 0.24"/>
+        </geometry>
+      </collision>
+      <inertial>
+        <origin xyz="0.06 0.0 0.095" rpy="0 0 0"/>
+        <mass value="20.656"/>
+        <inertia ixx="0.240" ixy="0.0" ixz="0.0" iyy="0.900" iyz="0.0" izz="1.050"/>
+      </inertial>
+    </xacro:if>
+    <xacro:unless value="$(arg simulation_physics)">
+      <inertial>
+        <origin xyz="0.064266 0.001648 0.095511" rpy="0 0 0"/>
+        <mass value="20.656"/>
+        <inertia ixx="0.110436033" ixy="0.007458962" ixz="-0.047319713" iyy="0.439622462" iyz="0.006320743" izz="0.625226807"/>
+      </inertial>
+    </xacro:unless>
   </link>
   <joint name="LeftWheel_joint" type="continuous">

File: amr_sweeper_description/urdf/sensors/IMU_sensor.xacro (robot description, xacro)
@@ -6,4 +6,24 @@
     <origin xyz="0.088 0.0 0.184" rpy="0 0 0"/>
   </joint>
-  <link name="imu_link"/>
+  <link name="imu_link">
+    <xacro:if value="$(arg simulation_physics)">
+      <visual>
+        <origin xyz="0 0 0" rpy="0 0 0"/>
+        <geometry>
+          <box size="0.02 0.02 0.01"/>
+        </geometry>
+      </visual>
+      <collision>
+        <origin xyz="0 0 0" rpy="0 0 0"/>
+        <geometry>
+          <box size="0.02 0.02 0.01"/>
+        </geometry>
+      </collision>
+      <inertial>
+        <origin xyz="0 0 0" rpy="0 0 0"/>
+        <mass value="0.05"/>
+        <inertia ixx="5.0e-6" ixy="0.0" ixz="0.0" iyy="5.0e-6" iyz="0.0" izz="5.0e-6"/>
+      </inertial>
+    </xacro:if>
+  </link>
 </robot>

File: amr_sweeper_description/urdf/sensors/depth_camera.xacro (robot description, xacro)
@@ -6,5 +6,13 @@
     <origin xyz="0.47 0 0.11" rpy="0 0 0"/>
   </joint>
-  <link name="realsense_mount"/>
+  <link name="realsense_mount">
+    <xacro:if value="$(arg simulation_physics)">
+      <inertial>
+        <origin xyz="0 0 0" rpy="0 0 0"/>
+        <mass value="0.02"/>
+        <inertia ixx="1.0e-5" ixy="0.0" ixz="0.0" iyy="1.0e-5" iyz="0.0" izz="1.0e-5"/>
+      </inertial>
+    </xacro:if>
+  </link>
   <joint name="realsense_mount_to_depth_camera_link" type="fixed">
     <parent link="realsense_mount"/>
@@ -12,5 +20,13 @@
     <origin xyz="0.015 0 -0.003" rpy="${pi} 0 0"/>
   </joint>
-  <link name="depth_camera_link"/>
+  <link name="depth_camera_link">
+    <xacro:if value="$(arg simulation_physics)">
+      <inertial>
+        <origin xyz="0 0 0" rpy="0 0 0"/>
+        <mass value="0.08"/>
+        <inertia ixx="2.0e-5" ixy="0.0" ixz="0.0" iyy="2.0e-5" iyz="0.0" izz="2.0e-5"/>
+      </inertial>
+    </xacro:if>
+  </link>
   <joint name="depth_camera_depth_frame_joint" type="fixed">
     <parent link="depth_camera_link"/>
